Commit message: v0.2.0 - Creation of segmented_cloud and inliers_indices messages and a segmented cloud coloring node

File: urdf/vision_test.xacro (robot description, xacro)
@@ -6,5 +6,5 @@
   <link name="base_link" />
   <link name="color"/>
-  <link name="realsense_rs200">
+  <link name="realsense_rs200">catkin_male
     <visual>
       <base_link rpy="0 0 0" xyz="0 0 0"/>
@@ -29,5 +29,5 @@
     <parent link="base_link" />
     <child link="color" />
-    <origin xyz="0 0 1.6" rpy="-2.09979 0.0 -1.57"/>
+    <origin xyz="0 -0.046 1.5004 " rpy="-2.070796 0 -1.570796"/>
   </joint>
 </robot>

Commit message: v0.2.5 Euclidian sementator

File: urdf/vision_test.xacro (robot description, xacro)
@@ -10,5 +10,5 @@
       <base_link rpy="0 0 0" xyz="0 0 0"/>
       <geometry>
-        <mesh filename="package://robot_eyes/meshes/realsense.dae"/>
+        <mesh filename="package://realsense_gazebo_plugin/models/realsense_camera/meshes/realsense.dae"/>
       </geometry>
     </visual>
